File: OneButton/Hardware/PCB/OneButton.sch (EAGLE design)
At the start: 36 parts, among them SW1 DHT-4235A, SW2 DHT-4235A, U1 WS2812, U10 STM32F042GU, U2 WS2812, U3 WS2812, U4 WS2812, U5 WS2812, U6 WS2812, U7 WS2812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

Commit message: Updated folder structure
Updated folder structure, adding software next
Parts:
- added Q1: BSS138W-7-F, OneButton:SMD-MOSFET-N-CH-50V-200MA-BSS138W-7-F(SOT-23)
- added R7, R8: 10k, OneButton:RESISTORRES-0603
Connections:
- removed net 5V: C14.1, C15.1, C2.1, J2.5, R2.2, R3.2, R4.2, U10MCU.VDDA, U10PWR.VDD@1, U9.OUT
- new net 3.3V: C14.1, C15.1, C2.1, J2.5, Q1.G, R2.2, R3.2, R4.2, R7.2, U10MCU.VDDA, U10PWR.VDD@1, U9.OUT
- new net N$2: Q1.S, R7.1, U10MCU.PB7
- net +5V: now also R8.2
- net DAT_IN: now also Q1.D, R8.1; no longer U10MCU.PB7
Other:
- note added: "2"
- note added: "2. LEVEL SHIFTER, 3.3V TO 5V. REQUIRED BY WS2812 FOR UNIPOLAR NZR COMMUNICATION 1. IN-LINE TERMINATION RESISTORS FOR USB 2.0, USB DP PULL-UP IS INTERNAL TO MCU NOTES: THIS PAGE"
- note removed: "1. IN-LINE TERMINATION RESISTORS FOR USB 2.0, USB DP PULL-UP IS INTERNAL TO MCU NOTES: THIS PAGE"
- moved on the sheet: C14, C15, U10
