File: Hardware/OneButton.sch (EAGLE design)
At the start: 39 parts, among them Q1 BSS138W-7-F, SW1 DHT-4235A, SW2 DHT-4235A, U1 WS2812, U10 STM32F042GU, U2 WS2812, U3 WS2812, U4 WS2812, U5 WS2812, U6 WS2812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

Commit message: CPP repo with working USB HID
CPP repo with working USB HID, thanks Andy!
Other:
- note added: "TODO: 1. Label SW-DEBUG port pins 2. Set BOOT0 to pull-down"
Changed lines of the file:
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@@
 <?xml version="1.0" encoding="utf-8"?>
 <!DOCTYPE eagle SYSTEM "eagle.dtd">
-<eagle version="8.4.3">
+<eagle version="8.5.0">
 <drawing>
 <settings>
@@
 <wire x1="360.68" y1="219.71" x2="368.3" y2="219.71" width="0.1524" layer="97"/>
 <wire x1="368.3" y1="219.71" x2="364.49" y2="226.06" width="0.1524" layer="97"/>
+<text x="236.22" y="139.7" size="1.778" layer="97">TODO:
+1.  Label SW-DEBUG port pins
+2. Set BOOT0 to pull-down</text>
 </plain>
 <instances>

Commit message: Working single button press
Remember to wait for the usb report to finish before sending the next
one!
Parts:
- C11: value DNP -> 0.1uF
- R2: value DNP -> 10k
Changed lines of the file:
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@@
 <part name="C10" library="OneButton" library_urn="urn:adsk.eagle:library:995496" deviceset="0.1UF" device="CAP-0603" package3d_urn="urn:adsk.eagle:package:1011647/2" value="0.1uF"/>
 <part name="R1" library="OneButton" library_urn="urn:adsk.eagle:library:995496" deviceset="RESISTOR" device="RES-0603" package3d_urn="urn:adsk.eagle:package:1000617/3" value="68R"/>
-<part name="R2" library="OneButton" library_urn="urn:adsk.eagle:library:995496" deviceset="RESISTOR" device="RES-0603" package3d_urn="urn:adsk.eagle:package:1000617/3" value="DNP"/>
+<part name="R2" library="OneButton" library_urn="urn:adsk.eagle:library:995496" deviceset="RESISTOR" device="RES-0603" package3d_urn="urn:adsk.eagle:package:1000617/3" value="10k"/>
 <part name="SUPPLY2" library="SparkFun-PowerSymbols" library_urn="urn:adsk.eagle:library:530" deviceset="3.3V" device=""/>
-<part name="C11" library="OneButton" library_urn="urn:adsk.eagle:library:995496" deviceset="CAPACITOR" device="CAP-0603" package3d_urn="urn:adsk.eagle:package:1011647/2" value="DNP"/>
+<part name="C11" library="OneButton" library_urn="urn:adsk.eagle:library:995496" deviceset="CAPACITOR" device="CAP-0603" package3d_urn="urn:adsk.eagle:package:1011647/2" value="0.1uF"/>
 <part name="SW1" library="OneButton" library_urn="urn:adsk.eagle:library:995496" deviceset="SMD-BUTTON-TOP-DHT-4235A(4P-4.2X3.2MM)" device="" package3d_urn="urn:adsk.eagle:package:1000734/2" value="DHT-4235A"/>
 <part name="GND5" library="supply1" library_urn="urn:adsk.eagle:library:371" deviceset="GND" device=""/>
