File: Hardware/OneButton.sch (EAGLE design)
At the start: 39 parts, among them Q1 BSS138W-7-F, SW1 DHT-4235A, SW2 DHT-4235A, U1 WS2812, U10 STM32F042GU, U2 WS2812, U3 WS2812, U4 WS2812, U5 WS2812, U6 WS2812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

Commit message: Code commit before creating ws8212 libs and adding cad files
Code commit before creating ws8212 libs and adding cad files
Other:
- note added: "TODO: 1. Label SW-DEBUG port pins 2. Set BOOT0 to pull-down 3. Move DAT_IN to SPI1 MOSI (PA7) 4. Move Button Pins and Button LED 5. Add surge current protection (IC)"
- note removed: "TODO: 1. Label SW-DEBUG port pins 2. Set BOOT0 to pull-down 3. Move DAT_IN to SPI1 MOSI (PA7) 4. Move Button Pins and Button LED"
Changed lines of the file:
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@@
 <?xml version="1.0" encoding="utf-8"?>
 <!DOCTYPE eagle SYSTEM "eagle.dtd">
-<eagle version="8.5.0">
+<eagle version="8.5.2">
 <drawing>
 <settings>
@@
 2. Set BOOT0 to pull-down
 3. Move DAT_IN to SPI1 MOSI (PA7)
-4. Move Button Pins and Button LED</text>
+4. Move Button Pins and Button LED
+5. Add surge current protection (IC)</text>
 </plain>
 <instances>

Commit message: Added debug instructions, removed build files
Added debug instructions, removed build files
Other:
- note added: "TODO: 1. Label SW-DEBUG port pins 2. Set BOOT0 to pull-down 3. Move DAT_IN to SPI1 MOSI (PA7) 4. Move Button Pins and Button LED 5. Add inrush current protection (IC)"
- note removed: "TODO: 1. Label SW-DEBUG port pins 2. Set BOOT0 to pull-down 3. Move DAT_IN to SPI1 MOSI (PA7) 4. Move Button Pins and Button LED 5. Add surge current protection (IC)"
Changed lines of the file:
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@@
 3. Move DAT_IN to SPI1 MOSI (PA7)
 4. Move Button Pins and Button LED
-5. Add surge current protection (IC)</text>
+5. Add inrush current protection (IC)</text>
 </plain>
 <instances>

Commit message: Updated circuit diagram TODOs and Firmware
Discovered that the board needs: 500mA current limiter circuit at the USB power input, 470R inline with DAT-IN, 1k between +5V and VCC, and about 200-1000uF more capacitance on +5V bus.
Other:
- note added: "TODO: 1. Label SW-DEBUG port pins 2. Set BOOT0 to pull-down 3. Move DAT_IN to SPI1 MOSI (PA7) 4. Move Button Pins and Button LED 5. Add inrush current protection (IC) 6. Add 150R between +5V and VCC, apply +5V directly to VDD. 7. Add 1000uF of capacitance to +5V bus"
- note removed: "TODO: 1. Label SW-DEBUG port pins 2. Set BOOT0 to pull-down 3. Move DAT_IN to SPI1 MOSI (PA7) 4. Move Button Pins and Button LED 5. Add inrush current protection (IC)"
Changed lines of the file:
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@@
 <?xml version="1.0" encoding="utf-8"?>
 <!DOCTYPE eagle SYSTEM "eagle.dtd">
-<eagle version="8.5.2">
+<eagle version="9.1.3">
 <drawing>
 <settings>
@@
 3. Move DAT_IN to SPI1 MOSI (PA7)
 4. Move Button Pins and Button LED
-5. Add inrush current protection (IC)</text>
+5. Add inrush current protection (IC)
+6. Add 150R between +5V and VCC, apply +5V directly to VDD.
+7. Add 1000uF of capacitance to +5V bus</text>
 </plain>
 <instances>
