File: Hardware/OneButton.brd (EAGLE design)
At the start: 50.8 x 50.8 mm, 39 parts, among them Q1 BSS138W-7-F, SW1 DHT-4235A, SW2 DHT-4235A, U1 WS2812, U10 STM32F042GU, U2 WS2812, U3 WS2812, U4 WS2812, U5 WS2812, U6 WS2812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

Commit message: Working single button press
Remember to wait for the usb report to finish before sending the next
one!
Parts:
- C11: value DNP -> 0.1uF
- R2: value DNP -> 10k
Changed lines of the file:
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@@
 <attribute name="NAME" x="19.558" y="11.43" size="0.8128" layer="25" font="vector" ratio="20" rot="R90" align="bottom-center"/>
 </element>
-<element name="R2" library="OneButton" library_urn="urn:adsk.eagle:library:995496" package="RESC0603_N" package3d_urn="urn:adsk.eagle:package:1000617/3" value="DNP" x="17.399" y="14.224" smashed="yes" rot="R270">
+<element name="R2" library="OneButton" library_urn="urn:adsk.eagle:library:995496" package="RESC0603_N" package3d_urn="urn:adsk.eagle:package:1000617/3" value="10k" x="17.399" y="14.224" smashed="yes" rot="R270">
 <attribute name="NAME" x="17.653" y="11.43" size="0.8128" layer="25" font="vector" ratio="20" rot="R90" align="bottom-center"/>
 </element>
-<element name="C11" library="OneButton" library_urn="urn:adsk.eagle:library:995496" package="CAP-0603" package3d_urn="urn:adsk.eagle:package:1011647/2" value="DNP" x="15.494" y="14.224" smashed="yes" rot="R270">
+<element name="C11" library="OneButton" library_urn="urn:adsk.eagle:library:995496" package="CAP-0603" package3d_urn="urn:adsk.eagle:package:1011647/2" value="0.1uF" x="15.494" y="14.224" smashed="yes" rot="R270">
 <attribute name="NAME" x="15.748" y="11.43" size="0.8128" layer="25" font="vector" ratio="20" rot="R90" align="bottom-center"/>
 </element>
